File: hardware/switchy_stamp_pth.brd (EAGLE design)
At the start: 38.1 x 25.4 mm, 23 parts, among them IC1 MC34063

Commit message: fixed a few mistakes, still rearranging
Other:
- board text added: "MK1.0"
Changed lines of the file:
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@@
 <?xml version="1.0" encoding="utf-8"?>
 <!DOCTYPE eagle SYSTEM "eagle.dtd">
-<eagle version="6.4">
+<eagle version="6.5.0">
 <drawing>
 <settings>
@@
 <wire x1="34.925" y1="25.4" x2="3.175" y2="25.4" width="0" layer="20"/>
 <wire x1="3.175" y1="25.4" x2="0" y2="22.225" width="0" layer="20" curve="90"/>
+<text x="29.21" y="23.876" size="1.016" layer="21" font="vector" ratio="12" align="bottom-center">MK1.0</text>
+<text x="28.956" y="23.876" size="1.016" layer="22" font="vector" ratio="12" rot="MR0" align="bottom-center">MK1.0</text>
 </plain>
 <attributes>
