File: hardware/switchy-stamp-buckeroo-mk-1.brd (EAGLE design)
At the start: 38.1 x 22.1 mm, 25 parts, among them IC1 MC34063

Commit message: more designfail
Parts:
- removed C4: 0.1uF, A_butts:C025-024X044
- removed IC1: MC34063, A_butts:DIP-08
- removed ON/OFF: SWITCH-SPDTSSA-12, A_butts:SWITCH-SPDT-SSA-12
- removed OUT: M02JST-PTH-2, A_butts:JST-2-PH-RA-PTH
- removed PWR: LED3MM, A_butts:LED3MM
- removed R2: 300R, A_butts:RESISTOR-AXIAL-PTH-5.08MM
- added CX2: 4.7uF@400V, A_butts:XC10B5
- added IC2: LNK306DIP-07, A_butts:DIP-07
- added L2: 1mH, A_butts:INDUCTOR-AXIAL-PTH-10.16MM
- C1: value 100uF -> 0.1uF; device A_butts:E2,5-7 -> A_butts:C025-024X044
- C2: value 470uF -> 100uF; device A_butts:E2,5-7 -> A_butts:E3,5-8
- C3: value 470pF -> 10uF; device A_butts:C025-024X044 -> A_butts:E3,5-8
- CX1: value (none) -> 4.7uF@400V
- D1: value 1N4001 -> 1N5819
- F1: value PTCPTH -> 1A; device A_butts:PTC -> A_butts:FUSE-2AG
- L1: value 220uH -> 1mH; device A_butts:RADIAL-PTH-6MMDIA -> A_butts:INDUCTOR-AXIAL-PTH-10.16MM
- R1: value 100R -> 13k; device A_butts:RESISTOR-AXIAL-PTH-5.08MM -> A_butts:RESISTOR-AXIAL-PTH-6.35MM
- R3: value 0.33R -> 2.05k; device A_butts:RESISTOR-AXIAL-PTH-10.16MM -> A_butts:RESISTOR-AXIAL-PTH-6.35MM
- R4: value 330R -> 3.3k; device A_butts:RESISTOR-AXIAL-PTH-5.08MM -> A_butts:RESISTOR-AXIAL-PTH-6.35MM
- moved D1 132.6 mm to (2.29, -123.7), turned to 0 degrees
- moved D2 131.6 mm to (2.29, -126.7)
- moved R3 129.6 mm to (1.27, -120.4), turned to 0 degrees
- moved R4 129.1 mm to (1.27, -117.3), turned to 0 degrees
- moved C3 127.5 mm to (0.25, -111.3), turned to 0 degrees
- moved C1 124.9 mm to (-0.76, -105.4), turned to 0 degrees
- moved C2 121.7 mm to (0.25, -99.3), turned to 0 degrees
- moved R1 98.7 mm to (1.27, -79.5)
- moved L1 88.1 mm to (3.05, -76.5)
- moved F1 84.6 mm to (9.91, -67.3), turned to 0 degrees
Connections:
- removed net GND: C1.-, C2.-, C3.2, C4.2, D2.A, IC1.4, OUT.2, R1.P$1, R4.P$1
- removed net N$12: B1.AC2, F1.P$1
- removed net N$3: IC1.5, R1.P$2, R2.P$1
- removed net N$5: C1.+, D1.C, IC1.6, R3.P$1
- removed net N$6: D2.C, IC1.2, L1.1
- removed net N$7: PWR.K, R4.P$2
- removed net N$9: B1.-
- removed net VOUT-: C2.+, C4.1, L1.2, OUT.1, PWR.A, R2.P$2
- new net 0V: B1.-, C2.-, CX1.2, CX2.2, D1.A, R4.P$1
- new net 12V: C2.+, D2.A, L1.P$2, R4.P$2
- new net N$13: CX2.1, IC2.5, L2.P$2
- new net N$14: C1.1, C3.-, D1.C, IC2.1, IC2.2, IC2.7, IC2.8, L1.P$1, R3.P$2
- new net N$15: C1.2, IC2.3
- net N$1: now also IC2.4, R1.P$1, R3.P$1; no longer IC1.1, IC1.7, IC1.8, R3.P$2
- net N$10: now also CX1.1, L2.P$1
- net N$11: now also B1.AC2; no longer F1.P$2
- net N$2: now also C3.+, D2.C, R1.P$2; no longer C3.1, IC1.3
- net N$4: now also F1.2, F1.2@2; no longer ON/OFF.B
- net N$8: now also F1.1, F1.1@1; no longer ON/OFF.COM
Routing:
- net VOUT-: track 27.6 -> 0.00 mm
- net N$5: track 18.9 -> 0.00 mm
- net N$1: track 14.8 -> 0.00 mm
- net N$3: track 10.3 -> 0.00 mm
- net N$6: track 8.17 -> 0.00 mm
- net N$7: track 4.06 -> 0.00 mm
- net N$2: track 2.90 -> 0.00 mm
- added copper zone on layer 1, net 0V
- removed copper zone on layer 1, net GND
