File: hardware/switchy-stamp-buckeroo-mk-1.sch (EAGLE design)
At the start: 23 parts, among them IC1 MC34063

Commit message: more designfail
Parts:
- removed C4: 0.1uF, A_butts:CAPACITOR-CERAMIC025-024X044
- removed IC1: MC34063, A_butts:MC34063DIP
- removed ON/OFF: SWITCH-SPDTSSA-12, A_butts:SWITCH-SPDTSSA-12
- removed OUT: M02JST-PTH-2, A_butts:M02JST-PTH-2
- removed PWR: LED3MM, A_butts:LED3MM
- removed R2: 300R, A_butts:RESISTORPTH-AXIAL-5.08MM
- added CX2: 4.7uF@400V, A_butts:CXXC10B5
- added IC2: LNK306DIP-07, A_butts:LNK306DIP-07
- added L2: 1mH, A_butts:INDUCTORAXIAL-PTH-10.16MM
- C1: value 100uF -> 0.1uF; device A_butts:CAPACITOR-POLARIZEDE2.5-7 -> A_butts:CAPACITOR-CERAMIC025-024X044
- C2: value 470uF -> 100uF; device A_butts:CAPACITOR-POLARIZEDE2.5-7 -> A_butts:CAPACITOR-POLARIZEDE3.5-8
- C3: value 470pF -> 10uF; device A_butts:CAPACITOR-CERAMIC025-024X044 -> A_butts:CAPACITOR-POLARIZEDE3.5-8
- CX1: value (none) -> 4.7uF@400V
- D1: value 1N4001 -> 1N5819; device A_butts:DIODEPTH-10.68MM -> A_butts:DIODE-SCHOTTKYPTH-10.16MM
- F1: value PTCPTH -> 1A; device A_butts:PTCPTH -> A_butts:FUSE5X20MM-2
- L1: value 220uH -> 1mH; device A_butts:INDUCTORPTH-RADIAL-6MMDIA -> A_butts:INDUCTORAXIAL-PTH-10.16MM
- R1: value 100R -> 13k; device A_butts:RESISTORPTH-AXIAL-5.08MM -> A_butts:RESISTORPTH-AXIAL-6.35MM
- R3: value 0.33R -> 2.05k; device A_butts:RESISTORPTH-AXIAL-10.16MM -> A_butts:RESISTORPTH-AXIAL-6.35MM
- R4: value 330R -> 3.3k; device A_butts:RESISTORPTH-AXIAL-5.08MM -> A_butts:RESISTORPTH-AXIAL-6.35MM
Connections:
- removed net GND: C1.-, C2.-, C3.2, C4.2, D2.A, IC1.GND, OUT.2, R1.1, R4.1
- removed net N$12: B1.AC2, F1.1
- removed net N$3: IC1.COMP, R1.2, R2.1
- removed net N$5: C1.+, D1.C, IC1.VCC, R3.1
- removed net N$6: D2.C, IC1.SWE, L1.1
- removed net N$7: PWR.C, R4.2
- removed net N$9: B1.-
- removed net VOUT-: C2.+, C4.1, L1.2, OUT.1, PWR.A, R2.2
- new net 0V: B1.-, C2.-, CX1.2, CX2.2, D1.A, R4.1
- new net 12V: C2.+, D2.A, L1.2, R4.2
- new net N$13: CX2.1, IC2.D, L2.2
- new net N$14: C1.1, C3.-, D1.C, IC2.S, L1.1, R3.2
- new net N$15: C1.2, IC2.BP
- net N$1: now also IC2.FB, R1.1, R3.1; no longer IC1.DVR, IC1.SEN, IC1.SWC, R3.2
- net N$10: now also CX1.1, L2.1
- net N$11: now also B1.AC2; no longer F1.2
- net N$2: now also C3.+, D2.C, R1.2; no longer C3.1, IC1.TC
- net N$4: now also F1.2; no longer ON/OFF.NO
- net N$8: now also F1.1; no longer ON/OFF.COM
Other:
- note added: "Offline Step-Down/Buck (85-265VAC to 5VDC)"
- note removed: "Step-Down/Buck (5V)"
- moved on the sheet: AC_IN, C2, CX1, D2, L1, R1, R3, R4
